Commit message: feat: integrate simplified EL-A3 gripper

File: el_a3_ros/el_a3_description/urdf/el_a3.urdf (robot description, URDF)
Before this commit: robot EL-A3, 10 links, 9 joints
Links:
- removed link gripper_link
- added link gripper_base_link, mass 0.180; collision box size=0.050 0.191 0.069; visual mesh filename=package://el_a3_description/meshes/gripper/visual/gripper_b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
- added link gripper_driver_link, mass 0.020; collision box size=0.008 0.008 0.016
- added link left_jaw_link, mass 0.035; collision box size=0.042 0.036 0.087; visual mesh filename=package://el_a3_description/meshes/gripper/visual/left_jaw_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
- added link right_jaw_link, mass 0.035; collision box size=0.042 0.036 0.087; visual mesh filename=package://el_a3_description/meshes/gripper/visual/right_jaw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
- link l5_l6_urdf_asm: geometry collision mesh filename=package://el_a3_description/meshes/el05_l6.stl; visual mesh filename=package://el_a3_description/meshes/el05_l6.stl
Joints:
- added joint gripper_base_joint: type fixed, parent l5_l6_urdf_asm, child gripper_base_link, origin xyz=0 0 0 rpy=0 0 0
- added joint left_jaw_joint: type prismatic, parent gripper_base_link, child left_jaw_link, origin xyz=0 0 0 rpy=0 0 0, axis 0 -1 0, limit lower=0 upper=0.05 effort=40 velocity=0.20, mimic joint=L7_joint multiplier=-0.031831 offset=0.05
- added joint right_jaw_joint: type prismatic, parent gripper_base_link, child right_jaw_link, origin xyz=0 0 0 rpy=0 0 0, axis 0 1 0, limit lower=0 upper=0.05 effort=40 velocity=0.20, mimic joint=L7_joint multiplier=-0.031831 offset=0.05
- joint L7_joint: child gripper_link -> gripper_driver_link; limit lower=-1.5708 upper=1.5708 effort=6.0 velocity=50 -> lower=0 upper=1.5708 effort=6.0 velocity=50

File: el_a3_ros/el_a3_description/urdf/el_a3.urdf.xacro (robot description, xacro)
@@ -8,4 +8,5 @@
   <xacro:arg name="host_can_id" default="253"/>
   <xacro:arg name="wrist_motor_type" default="EL05"/>
+  <xacro:arg name="use_gazebo" default="false"/>
   <!-- Wrist motor parameters (EL05: 6Nm, RS05: 5.5Nm) -->
   <xacro:property name="wrist_motor_type" value="$(arg wrist_motor_type)"/>
@@ -181,18 +182,4 @@
       </geometry>
     </collision>
-    <!-- Part jaw -->
-    <visual>
-      <origin xyz="0 0 -0.0755" rpy="3.14159 0 0"/>
-      <geometry>
-        <mesh filename="package://el_a3_description/meshes/jaw.stl"/>
-      </geometry>
-      <material name="orange"/>
-    </visual>
-    <collision>
-      <origin xyz="0 0 -0.0755" rpy="3.14159 0 0"/>
-      <geometry>
-        <mesh filename="package://el_a3_description/meshes/jaw.stl"/>
-      </geometry>
-    </collision>
   </link>
   <!-- End Effector link -->
@@ -259,20 +246,186 @@
     <child link="end_effector"/>
   </joint>
-  <!-- Joint L7 (${wrist_motor_type} Motor 7 - Gripper, separate kinematic branch) -->
+  <!--
+    L7 remains the physical gripper motor interface.  Its child is deliberately
+    invisible: the visible gripper is fixed to L6 and the two jaws mimic L7.
+    This preserves the controller, MoveIt, and joint_states interface while
+    preventing the gripper housing from rotating with the motor.
+  -->
   <joint name="L7_joint" type="revolute">
     <origin xyz="0 0 -0.074" rpy="0 0 0"/>
     <parent link="l5_l6_urdf_asm"/>
-    <child link="gripper_link"/>
-    <axis xyz="0 0 1"/>
-    <limit effort="${wrist_effort}" velocity="50" lower="-1.5708" upper="1.5708"/>
-    <dynamics damping="0.05" friction="0.05"/>
-  </joint>
-  <link name="gripper_link">
-    <inertial>
-      <mass value="0.05"/>
-      <origin xyz="0 0 0"/>
-      <inertia ixx="0.0001" ixy="0" ixz="0" iyy="0.0001" iyz="0" izz="0.0001"/>
-    </inertial>
-  </link>
+    <child link="gripper_driver_link"/>
+    <!-- Gazebo's imported wrist frame is mirrored relative to the CAD frame. -->
+    <xacro:if value="$(arg use_gazebo)">
+      <axis xyz="0 0 -1"/>
+    </xacro:if>
+    <xacro:unless value="$(arg use_gazebo)">
+      <axis xyz="0 0 1"/>
+    </xacro:unless>
+    <!-- 0 rad = closed, 1.5708 rad = open. -->
+    <limit effort="${wrist_effort}" velocity="50" lower="0" upper="1.5708"/>
+    <xacro:if value="$(arg use_gazebo)">
+      <dynamics damping="0" friction="0"/>
+    </xacro:if>
+    <xacro:unless value="$(arg use_gazebo)">
+      <dynamics damping="0.05" friction="0.05"/>
+    </xacro:unless>
+  </joint>
+  <link name="gripper_driver_link">
+    <inertial>
+      <mass value="0.020"/>
+      <!-- Offset from the fixed gripper base so Gazebo has no self-contact. -->
+      <origin xyz="0.040 0 -0.030"/>
+      <inertia ixx="2e-6" ixy="0" ixz="0" iyy="3.4e-5" iyz="0" izz="3.4e-5"/>
+    </inertial>
+    <!-- Collision-only body keeps the invisible L7 branch physical in Gazebo. -->
+    <collision>
+      <origin xyz="0.040 0 -0.030" rpy="0 0 0"/>
+      <geometry>
+        <box size="0.008 0.008 0.016"/>
+      </geometry>
+    </collision>
+  </link>
+  <!--
+    Simplified parallel gripper.  The supplied CAD meshes have X as the
+    approach axis, so a -90 degree Y rotation aligns them with the original
+    wrist/end-effector direction.  The base is on a fixed L6 branch; only the
+    lightweight driver link above rotates with L7.
+  -->
+  <joint name="gripper_base_joint" type="fixed">
+    <origin xyz="0 0 0" rpy="0 0 0"/>
+    <parent link="l5_l6_urdf_asm"/>
+    <child link="gripper_base_link"/>
+  </joint>
+  <link name="gripper_base_link">
+    <inertial>
+      <origin xyz="-0.1340 0 -0.1417" rpy="0 0 0"/>
+      <mass value="0.180"/>
+      <inertia ixx="0.00070" ixy="0" ixz="0" iyy="0.00025" iyz="0" izz="0.00075"/>
+    </inertial>
+    <visual>
+      <origin xyz="0 0 0" rpy="0 -1.5708 0"/>
+      <geometry>
+        <mesh filename="package://el_a3_description/meshes/gripper/visual/gripper_base.stl"/>
+      </geometry>
+      <material name="dark_brown"/>
+    </visual>
+    <collision>
+      <origin xyz="-0.1340 0 -0.1417" rpy="0 0 0"/>
+      <geometry>
+        <!-- Keep Gazebo's simplified base collision clear of both sliding rails. -->
+        <xacro:if value="$(arg use_gazebo)">
+          <box size="0.050 0.040 0.069"/>
+        </xacro:if>
+        <xacro:unless value="$(arg use_gazebo)">
+          <box size="0.050 0.191 0.069"/>
+        </xacro:unless>
+      </geometry>
+    </collision>
+  </link>
+  <joint name="left_jaw_joint" type="prismatic">
+    <xacro:if value="$(arg use_gazebo)">
+      <origin xyz="0 -0.05 0" rpy="0 0 0"/>
+    </xacro:if>
+    <xacro:unless value="$(arg use_gazebo)">
+      <origin xyz="0 0 0" rpy="0 0 0"/>
+    </xacro:unless>
+    <parent link="gripper_base_link"/>
+    <child link="left_jaw_link"/>
+    <!-- Positive motion is toward the gripper centre in the canonical URDF. -->
+    <xacro:if value="$(arg use_gazebo)">
+      <axis xyz="0 1 0"/>
+    </xacro:if>
+    <xacro:unless value="$(arg use_gazebo)">
+      <axis xyz="0 -1 0"/>
+    </xacro:unless>
+    <xacro:if value="$(arg use_gazebo)">
+      <limit effort="40" velocity="0.20" lower="0" upper="0.05"/>
+    </xacro:if>
+    <xacro:unless value="$(arg use_gazebo)">
+      <limit effort="40" velocity="0.20" lower="0" upper="0.05"/>
+    </xacro:unless>
+    <dynamics damping="5.0" friction="1.0"/>
+    <!-- Gazebo uses the ros2_control native mimic path (which has no offset). -->
+    <xacro:unless value="$(arg use_gazebo)">
+      <mimic joint="L7_joint" multiplier="-0.031831" offset="0.05"/>
+    </xacro:unless>
+  </joint>
+  <link name="left_jaw_link">
+    <inertial>
+      <origin xyz="-0.1342 0.0677 -0.2111" rpy="0 0 0"/>
+      <mass value="0.035"/>
+      <inertia ixx="0.000030" ixy="0" ixz="0" iyy="0.000030" iyz="0" izz="0.000020"/>
+    </inertial>
+    <visual>
+      <origin xyz="0 0 0" rpy="0 -1.5708 0"/>
+      <geometry>
+        <mesh filename="package://el_a3_description/meshes/gripper/visual/left_jaw_carriage.stl"/>
+      </geometry>
+      <material name="orange"/>
+    </visual>
+    <xacro:unless value="$(arg use_gazebo)">
+      <collision>
+        <origin xyz="-0.1342 0.0677 -0.2111" rpy="0 0 0"/>
+        <geometry>
+          <box size="0.042 0.036 0.087"/>
+        </geometry>
+      </collision>
+    </xacro:unless>
+  </link>
+  <joint name="right_jaw_joint" type="prismatic">
+    <xacro:if value="$(arg use_gazebo)">
+      <origin xyz="0 0.05 0" rpy="0 0 0"/>
+    </xacro:if>
+    <xacro:unless value="$(arg use_gazebo)">
+      <origin xyz="0 0 0" rpy="0 0 0"/>
+    </xacro:unless>
+    <parent link="gripper_base_link"/>
+    <child link="right_jaw_link"/>
+    <!-- Positive motion is toward the gripper centre. -->
+    <axis xyz="0 1 0"/>
+    <xacro:if value="$(arg use_gazebo)">
+      <limit effort="40" velocity="0.20" lower="-0.05" upper="0"/>
+    </xacro:if>
+    <xacro:unless value="$(arg use_gazebo)">
+      <limit effort="40" velocity="0.20" lower="0" upper="0.05"/>
+    </xacro:unless>
+    <dynamics damping="5.0" friction="1.0"/>
+    <!-- Gazebo uses the ros2_control native mimic path (which has no offset). -->
+    <xacro:unless value="$(arg use_gazebo)">
+      <mimic joint="L7_joint" multiplier="-0.031831" offset="0.05"/>
+    </xacro:unless>
+  </joint>
+  <link name="right_jaw_link">
+    <inertial>
+      <origin xyz="-0.1342 -0.0677 -0.2111" rpy="0 0 0"/>
+      <mass value="0.035"/>
+      <inertia ixx="0.000030" ixy="0" ixz="0" iyy="0.000030" iyz="0" izz="0.000020"/>
+    </inertial>
+    <visual>
+      <origin xyz="0 0 0" rpy="0 -1.5708 0"/>
+      <geometry>
+        <mesh filename="package://el_a3_description/meshes/gripper/visual/right_jaw_carriage.stl"/>
+      </geometry>
+      <material name="orange"/>
+    </visual>
+    <xacro:unless value="$(arg use_gazebo)">
+      <collision>
+        <origin xyz="-0.1342 -0.0677 -0.2111" rpy="0 0 0"/>
+        <geometry>
+          <box size="0.042 0.036 0.087"/>
+        </geometry>
+      </collision>
+    </xacro:unless>
+  </link>
+  <!-- Gazebo Sim uses the same L7 command interface and native mimic constraints. -->
+  <xacro:if value="$(arg use_gazebo)">
+    <gazebo>
+      <!-- Humble/Fortress exports the compatibility alias below from gz_ros2_control. -->
+      <plugin filename="gz_ros2_control-system" name="ign_ros2_control::IgnitionROS2ControlPlugin">
+        <parameters>$(find el_a3_description)/config/el_a3_controllers.yaml</parameters>
+      </plugin>
+    </gazebo>
+  </xacro:if>
   <!-- ros2_control interface -->
   <xacro:el_a3_ros2_control
@@ -280,4 +433,5 @@
     can_interface="$(arg can_interface)"
     host_can_id="$(arg host_can_id)"
-    wrist_motor_type="$(arg wrist_motor_type)"/>
+    wrist_motor_type="$(arg wrist_motor_type)"
+    use_gazebo="$(arg use_gazebo)"/>
 </robot>

File: el_a3_ros/el_a3_description/urdf/el_a3_ros2_control.xacro (robot description, xacro)
@@ -2,5 +2,5 @@
 <!-- EL-A3 ros2_control configuration -->
 <robot xmlns:xacro="http://www.ros.org/wiki/xacro">
-  <xacro:macro name="el_a3_ros2_control" params="use_mock_hardware can_interface host_can_id wrist_motor_type">
+  <xacro:macro name="el_a3_ros2_control" params="use_mock_hardware can_interface host_can_id wrist_motor_type use_gazebo">
     <!-- Wrist motor effort limits based on motor type -->
     <xacro:property name="wrist_effort_max" value="${5.5 if wrist_motor_type == 'RS05' else 6.0}"/>
@@ -8,9 +8,12 @@
     <ros2_control name="RsA3System" type="system">
       <hardware>
-        <xacro:if value="${use_mock_hardware}">
+        <xacro:if value="${use_gazebo}">
+          <plugin>gz_ros2_control/GazeboSimSystem</plugin>
+        </xacro:if>
+        <xacro:if value="${use_mock_hardware and not use_gazebo}">
           <plugin>mock_components/GenericSystem</plugin>
           <param name="mock_sensor_commands">false</param>
         </xacro:if>
-        <xacro:unless value="${use_mock_hardware}">
+        <xacro:if value="${not use_mock_hardware and not use_gazebo}">
           <plugin>el_a3_hardware/RsA3HardwareInterface</plugin>
           <param name="can_interface">${can_interface}</param>
@@ -73,5 +76,5 @@
           <param name="gravity_comp_L6_cos">0.0</param>
           <param name="gravity_comp_L6_offset">0.0</param>
-        </xacro:unless>
+        </xacro:if>
       </hardware>
       <!-- Joint L1 - RS00 Motor 1 -->
@@ -232,19 +235,35 @@
         <param name="zero_torque_kd_max">0.10</param>
         <command_interface name="position">
-          <param name="min">-1.5708</param>
-          <param name="max">1.5708</param>
-        </command_interface>
-        <command_interface name="velocity">
-          <param name="min">-50.0</param>
-          <param name="max">50.0</param>
-        </command_interface>
-        <command_interface name="effort">
-          <param name="min">${wrist_effort_min}</param>
-          <param name="max">${wrist_effort_max}</param>
-        </command_interface>
-        <state_interface name="position"/>
-        <state_interface name="velocity"/>
-        <state_interface name="effort"/>
-      </joint>
+          <param name="min">0</param>
+          <param name="max">1.5708</param>
+        </command_interface>
+        <command_interface name="velocity">
+          <param name="min">-50.0</param>
+          <param name="max">50.0</param>
+        </command_interface>
+        <command_interface name="effort">
+          <param name="min">${wrist_effort_min}</param>
+          <param name="max">${wrist_effort_max}</param>
+        </command_interface>
+        <state_interface name="position"/>
+        <state_interface name="velocity"/>
+        <state_interface name="effort"/>
+      </joint>
+      <!-- Gazebo's native mimic path; real hardware has only L7. -->
+      <xacro:if value="${use_gazebo}">
+        <joint name="left_jaw_joint">
+          <param name="mimic">L7_joint</param>
+          <!-- Gazebo uses a positive left rail axis; its zero is pre-shifted closed. -->
+          <param name="multiplier">0.031831</param>
+          <state_interface name="position"/>
+          <state_interface name="velocity"/>
+        </joint>
+        <joint name="right_jaw_joint">
+          <param name="mimic">L7_joint</param>
+          <param name="multiplier">-0.031831</param>
+          <state_interface name="position"/>
+          <state_interface name="velocity"/>
+        </joint>
+      </xacro:if>
     </ros2_control>
   </xacro:macro>
