Commit message: chore: remove Gazebo gripper integration

File: el_a3_ros/el_a3_description/urdf/el_a3.urdf (robot description, URDF)
Before this commit: robot EL-A3, 13 links, 12 joints
Links:
- link gripper_driver_link: geometry 

File: el_a3_ros/el_a3_description/urdf/el_a3.urdf.xacro (robot description, xacro)
@@ -8,5 +8,4 @@
   <xacro:arg name="host_can_id" default="253"/>
   <xacro:arg name="wrist_motor_type" default="EL05"/>
-  <xacro:arg name="use_gazebo" default="false"/>
   <!-- Wrist motor parameters (EL05: 6Nm, RS05: 5.5Nm) -->
   <xacro:property name="wrist_motor_type" value="$(arg wrist_motor_type)"/>
@@ -256,34 +255,15 @@
     <parent link="l5_l6_urdf_asm"/>
     <child link="gripper_driver_link"/>
-    <!-- Gazebo's imported wrist frame is mirrored relative to the CAD frame. -->
-    <xacro:if value="$(arg use_gazebo)">
-      <axis xyz="0 0 -1"/>
-    </xacro:if>
-    <xacro:unless value="$(arg use_gazebo)">
-      <axis xyz="0 0 1"/>
-    </xacro:unless>
+    <axis xyz="0 0 1"/>
     <!-- 0 rad = closed, 1.5708 rad = open. -->
     <limit effort="${wrist_effort}" velocity="50" lower="0" upper="1.5708"/>
-    <xacro:if value="$(arg use_gazebo)">
-      <dynamics damping="0" friction="0"/>
-    </xacro:if>
-    <xacro:unless value="$(arg use_gazebo)">
-      <dynamics damping="0.05" friction="0.05"/>
-    </xacro:unless>
+    <dynamics damping="0.05" friction="0.05"/>
   </joint>
   <link name="gripper_driver_link">
     <inertial>
       <mass value="0.020"/>
-      <!-- Offset from the fixed gripper base so Gazebo has no self-contact. -->
       <origin xyz="0.040 0 -0.030"/>
       <inertia ixx="2e-6" ixy="0" ixz="0" iyy="3.4e-5" iyz="0" izz="3.4e-5"/>
     </inertial>
-    <!-- Collision-only body keeps the invisible L7 branch physical in Gazebo. -->
-    <collision>
-      <origin xyz="0.040 0 -0.030" rpy="0 0 0"/>
-      <geometry>
-        <box size="0.008 0.008 0.016"/>
-      </geometry>
-    </collision>
   </link>
   <!--
@@ -314,41 +294,17 @@
       <origin xyz="-0.1340 0 -0.1417" rpy="0 0 0"/>
       <geometry>
-        <!-- Keep Gazebo's simplified base collision clear of both sliding rails. -->
-        <xacro:if value="$(arg use_gazebo)">
-          <box size="0.050 0.040 0.069"/>
-        </xacro:if>
-        <xacro:unless value="$(arg use_gazebo)">
-          <box size="0.050 0.191 0.069"/>
-        </xacro:unless>
+        <box size="0.050 0.191 0.069"/>
       </geometry>
     </collision>
   </link>
   <joint name="left_jaw_joint" type="prismatic">
-    <xacro:if value="$(arg use_gazebo)">
-      <origin xyz="0 -0.05 0" rpy="0 0 0"/>
-    </xacro:if>
-    <xacro:unless value="$(arg use_gazebo)">
-      <origin xyz="0 0 0" rpy="0 0 0"/>
-    </xacro:unless>
+    <origin xyz="0 0 0" rpy="0 0 0"/>
     <parent link="gripper_base_link"/>
     <child link="left_jaw_link"/>
-    <!-- Positive motion is toward the gripper centre in the canonical URDF. -->
-    <xacro:if value="$(arg use_gazebo)">
-      <axis xyz="0 1 0"/>
-    </xacro:if>
-    <xacro:unless value="$(arg use_gazebo)">
-      <axis xyz="0 -1 0"/>
-    </xacro:unless>
-    <xacro:if value="$(arg use_gazebo)">
-      <limit effort="40" velocity="0.20" lower="0" upper="0.05"/>
-    </xacro:if>
-    <xacro:unless value="$(arg use_gazebo)">
-      <limit effort="40" velocity="0.20" lower="0" upper="0.05"/>
-    </xacro:unless>
+    <!-- Positive motion is toward the gripper centre. -->
+    <axis xyz="0 -1 0"/>
+    <limit effort="40" velocity="0.20" lower="0" upper="0.05"/>
     <dynamics damping="5.0" friction="1.0"/>
-    <!-- Gazebo uses the ros2_control native mimic path (which has no offset). -->
-    <xacro:unless value="$(arg use_gazebo)">
-      <mimic joint="L7_joint" multiplier="-0.031831" offset="0.05"/>
-    </xacro:unless>
+    <mimic joint="L7_joint" multiplier="-0.031831" offset="0.05"/>
   </joint>
   <link name="left_jaw_link">
@@ -365,35 +321,20 @@
       <material name="orange"/>
     </visual>
-    <xacro:unless value="$(arg use_gazebo)">
-      <collision>
-        <origin xyz="-0.1342 0.0677 -0.2111" rpy="0 0 0"/>
-        <geometry>
-          <box size="0.042 0.036 0.087"/>
-        </geometry>
-      </collision>
-    </xacro:unless>
+    <collision>
+      <origin xyz="-0.1342 0.0677 -0.2111" rpy="0 0 0"/>
+      <geometry>
+        <box size="0.042 0.036 0.087"/>
+      </geometry>
+    </collision>
   </link>
   <joint name="right_jaw_joint" type="prismatic">
-    <xacro:if value="$(arg use_gazebo)">
-      <origin xyz="0 0.05 0" rpy="0 0 0"/>
-    </xacro:if>
-    <xacro:unless value="$(arg use_gazebo)">
-      <origin xyz="0 0 0" rpy="0 0 0"/>
-    </xacro:unless>
+    <origin xyz="0 0 0" rpy="0 0 0"/>
     <parent link="gripper_base_link"/>
     <child link="right_jaw_link"/>
     <!-- Positive motion is toward the gripper centre. -->
     <axis xyz="0 1 0"/>
-    <xacro:if value="$(arg use_gazebo)">
-      <limit effort="40" velocity="0.20" lower="-0.05" upper="0"/>
-    </xacro:if>
-    <xacro:unless value="$(arg use_gazebo)">
-      <limit effort="40" velocity="0.20" lower="0" upper="0.05"/>
-    </xacro:unless>
+    <limit effort="40" velocity="0.20" lower="0" upper="0.05"/>
     <dynamics damping="5.0" friction="1.0"/>
-    <!-- Gazebo uses the ros2_control native mimic path (which has no offset). -->
-    <xacro:unless value="$(arg use_gazebo)">
-      <mimic joint="L7_joint" multiplier="-0.031831" offset="0.05"/>
-    </xacro:unless>
+    <mimic joint="L7_joint" multiplier="-0.031831" offset="0.05"/>
   </joint>
   <link name="right_jaw_link">
@@ -410,22 +351,11 @@
       <material name="orange"/>
     </visual>
-    <xacro:unless value="$(arg use_gazebo)">
-      <collision>
-        <origin xyz="-0.1342 -0.0677 -0.2111" rpy="0 0 0"/>
-        <geometry>
-          <box size="0.042 0.036 0.087"/>
-        </geometry>
-      </collision>
-    </xacro:unless>
-  </link>
-  <!-- Gazebo Sim uses the same L7 command interface and native mimic constraints. -->
-  <xacro:if value="$(arg use_gazebo)">
-    <gazebo>
-      <!-- Humble/Fortress exports the compatibility alias below from gz_ros2_control. -->
-      <plugin filename="gz_ros2_control-system" name="ign_ros2_control::IgnitionROS2ControlPlugin">
-        <parameters>$(find el_a3_description)/config/el_a3_controllers.yaml</parameters>
-      </plugin>
-    </gazebo>
-  </xacro:if>
+    <collision>
+      <origin xyz="-0.1342 -0.0677 -0.2111" rpy="0 0 0"/>
+      <geometry>
+        <box size="0.042 0.036 0.087"/>
+      </geometry>
+    </collision>
+  </link>
   <!-- ros2_control interface -->
   <xacro:el_a3_ros2_control
@@ -433,5 +363,4 @@
     can_interface="$(arg can_interface)"
     host_can_id="$(arg host_can_id)"
-    wrist_motor_type="$(arg wrist_motor_type)"
-    use_gazebo="$(arg use_gazebo)"/>
+    wrist_motor_type="$(arg wrist_motor_type)"/>
 </robot>

File: el_a3_ros/el_a3_description/urdf/el_a3_ros2_control.xacro (robot description, xacro)
@@ -2,5 +2,5 @@
 <!-- EL-A3 ros2_control configuration -->
 <robot xmlns:xacro="http://www.ros.org/wiki/xacro">
-  <xacro:macro name="el_a3_ros2_control" params="use_mock_hardware can_interface host_can_id wrist_motor_type use_gazebo">
+  <xacro:macro name="el_a3_ros2_control" params="use_mock_hardware can_interface host_can_id wrist_motor_type">
     <!-- Wrist motor effort limits based on motor type -->
     <xacro:property name="wrist_effort_max" value="${5.5 if wrist_motor_type == 'RS05' else 6.0}"/>
@@ -8,12 +8,9 @@
     <ros2_control name="RsA3System" type="system">
       <hardware>
-        <xacro:if value="${use_gazebo}">
-          <plugin>gz_ros2_control/GazeboSimSystem</plugin>
-        </xacro:if>
-        <xacro:if value="${use_mock_hardware and not use_gazebo}">
+        <xacro:if value="${use_mock_hardware}">
           <plugin>mock_components/GenericSystem</plugin>
           <param name="mock_sensor_commands">false</param>
         </xacro:if>
-        <xacro:if value="${not use_mock_hardware and not use_gazebo}">
+        <xacro:unless value="${use_mock_hardware}">
           <plugin>el_a3_hardware/RsA3HardwareInterface</plugin>
           <param name="can_interface">${can_interface}</param>
@@ -76,5 +73,5 @@
           <param name="gravity_comp_L6_cos">0.0</param>
           <param name="gravity_comp_L6_offset">0.0</param>
-        </xacro:if>
+        </xacro:unless>
       </hardware>
       <!-- Joint L1 - RS00 Motor 1 -->
@@ -250,20 +247,4 @@
         <state_interface name="effort"/>
       </joint>
-      <!-- Gazebo's native mimic path; real hardware has only L7. -->
-      <xacro:if value="${use_gazebo}">
-        <joint name="left_jaw_joint">
-          <param name="mimic">L7_joint</param>
-          <!-- Gazebo uses a positive left rail axis; its zero is pre-shifted closed. -->
-          <param name="multiplier">0.031831</param>
-          <state_interface name="position"/>
-          <state_interface name="velocity"/>
-        </joint>
-        <joint name="right_jaw_joint">
-          <param name="mimic">L7_joint</param>
-          <param name="multiplier">-0.031831</param>
-          <state_interface name="position"/>
-          <state_interface name="velocity"/>
-        </joint>
-      </xacro:if>
     </ros2_control>
   </xacro:macro>

Commit message: fix: update gripper base mesh and collisions

File: el_a3_ros/el_a3_description/urdf/el_a3.urdf (robot description, URDF)
Before this commit: robot EL-A3, 13 links, 12 joints
Links:
- link gripper_base_link: geometry collision box size=0.050 0.040 0.012; visual mesh filename=package://el_a3_description/meshes/gripper/visual/gripper_b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
- link left_jaw_link: geometry collision box size=0.042 0.032 0.087; visual mesh filename=package://el_a3_description/meshes/gripper/visual/left_jaw_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
- link right_jaw_link: geometry collision box size=0.042 0.032 0.087; visual mesh filename=package://el_a3_description/meshes/gripper/visual/right_jaw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

File: el_a3_ros/el_a3_description/urdf/el_a3.urdf.xacro (robot description, xacro)
@@ -292,7 +292,8 @@
     </visual>
     <collision>
-      <origin xyz="-0.1340 0 -0.1417" rpy="0 0 0"/>
-      <geometry>
-        <box size="0.050 0.191 0.069"/>
+      <!-- Central mounting block only: keep both jaw slide paths collision-free. -->
+      <origin xyz="-0.1340 0 -0.1560" rpy="0 0 0"/>
+      <geometry>
+        <box size="0.050 0.040 0.012"/>
       </geometry>
     </collision>
@@ -324,5 +325,5 @@
       <origin xyz="-0.1342 0.0677 -0.2111" rpy="0 0 0"/>
       <geometry>
-        <box size="0.042 0.036 0.087"/>
+        <box size="0.042 0.032 0.087"/>
       </geometry>
     </collision>
@@ -354,5 +355,5 @@
       <origin xyz="-0.1342 -0.0677 -0.2111" rpy="0 0 0"/>
       <geometry>
-        <box size="0.042 0.036 0.087"/>
+        <box size="0.042 0.032 0.087"/>
       </geometry>
     </collision>

Commit message: fix: align gripper horizontally at wrist

File: el_a3_ros/el_a3_description/urdf/el_a3.urdf (robot description, URDF)
Before this commit: robot EL-A3, 13 links, 12 joints
Links:
- link gripper_base_link: geometry collision box size=0.040 0.050 0.012; visual mesh filename=package://el_a3_description/meshes/gripper/visual/gripper_b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
- link left_jaw_link: geometry collision box size=0.032 0.042 0.087; visual mesh filename=package://el_a3_description/meshes/gripper/visual/left_jaw_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
- link right_jaw_link: geometry collision box size=0.032 0.042 0.087; visual mesh filename=package://el_a3_description/meshes/gripper/visual/right_jaw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
Joints:
- joint left_jaw_joint: axis 0 -1 0 -> -1 0 0
- joint right_jaw_joint: axis 0 1 0 -> 1 0 0

File: el_a3_ros/el_a3_description/urdf/el_a3.urdf.xacro (robot description, xacro)
@@ -268,8 +268,9 @@
   </link>
   <!--
-    Simplified parallel gripper.  The supplied CAD meshes have X as the
-    approach axis, so a -90 degree Y rotation aligns them with the original
-    wrist/end-effector direction.  The base is on a fixed L6 branch; only the
-    lightweight driver link above rotates with L7.
+    Simplified parallel gripper. The supplied CAD meshes share a global CAD
+    frame: X is the approach axis and Y is the jaw span. Rotate that frame into
+    the wrist frame and compensate its CAD origin so the jaws span horizontally
+    across the end effector. The base is fixed to L6; only the lightweight
+    driver link above rotates with L7.
   -->
   <joint name="gripper_base_joint" type="fixed">
@@ -280,10 +281,10 @@
   <link name="gripper_base_link">
     <inertial>
-      <origin xyz="-0.1340 0 -0.1417" rpy="0 0 0"/>
+      <origin xyz="0 0 -0.1636" rpy="0 0 0"/>
       <mass value="0.180"/>
-      <inertia ixx="0.00070" ixy="0" ixz="0" iyy="0.00025" iyz="0" izz="0.00075"/>
-    </inertial>
-    <visual>
-      <origin xyz="0 0 0" rpy="0 -1.5708 0"/>
+      <inertia ixx="0.00025" ixy="0" ixz="0" iyy="0.00070" iyz="0" izz="0.00075"/>
+    </inertial>
+    <visual>
+      <origin xyz="0 -0.1340 0" rpy="0 -1.5708 -1.5708"/>
       <geometry>
         <mesh filename="package://el_a3_description/meshes/gripper/visual/gripper_base.stl"/>
@@ -293,7 +294,7 @@
     <collision>
       <!-- Central mounting block only: keep both jaw slide paths collision-free. -->
-      <origin xyz="-0.1340 0 -0.1560" rpy="0 0 0"/>
-      <geometry>
-        <box size="0.050 0.040 0.012"/>
+      <origin xyz="0 0 -0.1560" rpy="0 0 0"/>
+      <geometry>
+        <box size="0.040 0.050 0.012"/>
       </geometry>
     </collision>
@@ -304,5 +305,5 @@
     <child link="left_jaw_link"/>
     <!-- Positive motion is toward the gripper centre. -->
-    <axis xyz="0 -1 0"/>
+    <axis xyz="-1 0 0"/>
     <limit effort="40" velocity="0.20" lower="0" upper="0.05"/>
     <dynamics damping="5.0" friction="1.0"/>
@@ -311,10 +312,10 @@
   <link name="left_jaw_link">
     <inertial>
-      <origin xyz="-0.1342 0.0677 -0.2111" rpy="0 0 0"/>
+      <origin xyz="0.0677 0.0003 -0.2111" rpy="0 0 0"/>
       <mass value="0.035"/>
       <inertia ixx="0.000030" ixy="0" ixz="0" iyy="0.000030" iyz="0" izz="0.000020"/>
     </inertial>
     <visual>
-      <origin xyz="0 0 0" rpy="0 -1.5708 0"/>
+      <origin xyz="0 -0.1340 0" rpy="0 -1.5708 -1.5708"/>
       <geometry>
         <mesh filename="package://el_a3_description/meshes/gripper/visual/left_jaw_carriage.stl"/>
@@ -323,7 +324,7 @@
     </visual>
     <collision>
-      <origin xyz="-0.1342 0.0677 -0.2111" rpy="0 0 0"/>
-      <geometry>
-        <box size="0.042 0.032 0.087"/>
+      <origin xyz="0.0677 0.0003 -0.2111" rpy="0 0 0"/>
+      <geometry>
+        <box size="0.032 0.042 0.087"/>
       </geometry>
     </collision>
@@ -334,5 +335,5 @@
     <child link="right_jaw_link"/>
     <!-- Positive motion is toward the gripper centre. -->
-    <axis xyz="0 1 0"/>
+    <axis xyz="1 0 0"/>
     <limit effort="40" velocity="0.20" lower="0" upper="0.05"/>
     <dynamics damping="5.0" friction="1.0"/>
@@ -341,10 +342,10 @@
   <link name="right_jaw_link">
     <inertial>
-      <origin xyz="-0.1342 -0.0677 -0.2111" rpy="0 0 0"/>
+      <origin xyz="-0.0677 0.0003 -0.2111" rpy="0 0 0"/>
       <mass value="0.035"/>
       <inertia ixx="0.000030" ixy="0" ixz="0" iyy="0.000030" iyz="0" izz="0.000020"/>
     </inertial>
     <visual>
-      <origin xyz="0 0 0" rpy="0 -1.5708 0"/>
+      <origin xyz="0 -0.1340 0" rpy="0 -1.5708 -1.5708"/>
       <geometry>
         <mesh filename="package://el_a3_description/meshes/gripper/visual/right_jaw_carriage.stl"/>
@@ -353,7 +354,7 @@
     </visual>
     <collision>
-      <origin xyz="-0.1342 -0.0677 -0.2111" rpy="0 0 0"/>
-      <geometry>
-        <box size="0.042 0.032 0.087"/>
+      <origin xyz="-0.0677 0.0003 -0.2111" rpy="0 0 0"/>
+      <geometry>
+        <box size="0.032 0.042 0.087"/>
       </geometry>
     </collision>

Commit message: fix: mount gripper at wrist flange

File: el_a3_ros/el_a3_description/urdf/el_a3.urdf (robot description, URDF)
Before this commit: robot EL-A3, 13 links, 12 joints
Joints:
- joint gripper_base_joint: origin xyz=0 0 0 rpy=0 0 0 -> xyz=0 0 0.045 rpy=0 0 0

File: el_a3_ros/el_a3_description/urdf/el_a3.urdf.xacro (robot description, xacro)
@@ -275,5 +275,6 @@
   -->
   <joint name="gripper_base_joint" type="fixed">
-    <origin xyz="0 0 0" rpy="0 0 0"/>
+    <!-- Match the wrist flange plane used by the original jaw mesh. -->
+    <origin xyz="0 0 0.045" rpy="0 0 0"/>
     <parent link="l5_l6_urdf_asm"/>
     <child link="gripper_base_link"/>
